File: Hardware/SparkFun NEO-M8T.brd (EAGLE design)
At the start: 40.6 x 33 mm, 94 parts, among them J13 U.FL, J2 Qwiic Right Angle, J4 Qwiic Right Angle, U1 U-BLOX_NEO-M9N, U2 3.3V

Commit message: Some updates to the design (heh)
Parts:
- removed U$2: (no value), board lables:NEO#M9N1
- JP15: device SparkFun-Connectors:1X04_NO_SILK -> SparkFun-Connectors:1X05_NO_SILK
- U1: value U-BLOX_NEO-M9N -> U-BLOX_NEO-M8T; device SparkFun-GPS:NEO-M9N -> SparkFun-GPS:NEO-M9N/M8T
- moved U$35 2.54 mm to (14.0, 1.40)
- moved U$36 2.54 mm to (14.0, 1.40)
- moved U$43 2.54 mm to (11.4, 1.65)
- moved U$44 2.54 mm to (11.4, 1.65)
- moved U$39 2.54 mm to (16.5, 1.40)
- moved U$40 2.54 mm to (16.5, 1.40)
Connections:
- net SCL_LV renamed N$13
- net SDA_LV renamed N$3
- removed net !SAFE: JP15.2, U1.1
- removed net INT: JP15.1, U1.4
- new net INT0: JP15.2, U1.4
- new net INT1: JP15.1, U1.15
- new net TP2/!SAFE: JP15.3, U1.1
- net !RESET: now also JP15.4; no longer JP15.3
- net PPS: now also JP15.5; no longer JP15.4
Routing:
- net INT: track 23.7 -> 0.00 mm, vias 1 -> 0
- net INT0: track 0.00 -> 21.5 mm, vias 0 -> 1
- net !SAFE: track 17.9 -> 0.00 mm, vias 1 -> 0
- net TP2/!SAFE: track 0.00 -> 15.3 mm, vias 0 -> 1
- net N$3: track 4.00 -> 0.00 mm
- net N$13: track 3.83 -> 0.00 mm
- net PPS: track 36.8 -> 33.2 mm
- net !RESET: track 27.9 -> 24.7 mm
- removed copper zone on layer 1, net GPS_ANT1

Commit message: Removes 10k from board
Parts:
- removed R16: 10k, SparkFun-Resistors:0402
Connections:
- net 3.3V: no longer R16.2
- net D_SEL: no longer R16.1
Routing:
- net PPS: track 33.2 -> 23.6 mm
- net !RESET: track 24.7 -> 16.9 mm
- net TP2/!SAFE: track 15.3 -> 9.35 mm
- net INT0: track 21.5 -> 17.6 mm
- net 3.3V: track 109.6 -> 108.2 mm, vias 8 -> 7
- net D_SEL: track 4.85 -> 3.95 mm
- net GND: vias 170 -> 169
Changed lines of the file:
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@@
 <layer number="19" name="Unrouted" color="6" fill="1" visible="yes" active="yes"/>
 <layer number="20" name="Dimension" color="15" fill="1" visible="yes" active="yes"/>
-<layer number="21" name="tPlace" color="16" fill="1" visible="yes" active="yes"/>
-<layer number="22" name="bPlace" color="14" fill="1" visible="yes" active="yes"/>
+<layer number="21" name="tPlace" color="16" fill="1" visible="no" active="yes"/>
+<layer number="22" name="bPlace" color="14" fill="1" visible="no" active="yes"/>
 <layer number="23" name="tOrigins" color="15" fill="1" visible="yes" active="yes"/>
 <layer number="24" name="bOrigins" color="15" fill="1" visible="yes" active="yes"/>
@@
 <attribute name="VALUE" x="6.858" y="22.8346" size="0.6096" layer="27" font="vector" ratio="20" rot="R90" align="top-center"/>
 </element>
-<element name="R16" library="SparkFun-Resistors" package="0402" value="10k" x="29.718" y="10.414" smashed="yes" rot="R270">
-<attribute name="NAME" x="30.48" y="10.414" size="0.6096" layer="25" font="vector" ratio="20" rot="R270" align="bottom-center"/>
-<attribute name="PROD_ID" value="RES-14241" x="29.718" y="10.414" size="1.778" layer="27" font="vector" rot="R270" display="off"/>
-<attribute name="VALUE" x="28.956" y="10.414" size="0.6096" layer="27" font="vector" ratio="20" rot="R270" align="top-center"/>
-</element>
 <element name="U$11" library="board lables" package="SPI1" value="" x="30.734" y="7.62" smashed="yes" rot="MR0"/>
 <element name="U$13" library="SparkFun-Aesthetics" package="QWIIC_4MM" value="" x="38.354" y="20.574" smashed="yes"/>
@@
 <wire x1="5.08" y1="20.574" x2="5.08" y2="18.0006" width="0.508" layer="16"/>
 <wire x1="5.97123125" y1="20.574" x2="5.08" y2="20.574" width="0.508" layer="16"/>
-<wire x1="5.97123125" y1="20.574" x2="10.859615625" y2="25.462384375" width="0.508" layer="16"/>
-<contactref element="R16" pad="2"/>
-<wire x1="10.859615625" y1="25.462384375" x2="11.68623125" y2="26.289" width="0.508" layer="16"/>
-<wire x1="29.718" y1="9.834" x2="29.845" y2="9.707" width="0.508" layer="1"/>
-<wire x1="29.845" y1="9.707" x2="29.845" y2="8.4836" width="0.508" layer="1"/>
-<via x="29.845" y="8.4836" extent="1-16" drill="0.3048"/>
+<wire x1="5.97123125" y1="20.574" x2="11.68623125" y2="26.289" width="0.508" layer="16"/>
 <wire x1="11.68623125" y1="26.289" x2="15.367" y2="26.289" width="0.508" layer="16"/>
 <wire x1="15.9766" y1="26.8986" x2="17.145" y2="26.8986" width="0.508" layer="16"/>
@@
 <via x="33.782" y="6.3246" extent="1-16" drill="0.3048"/>
 <via x="8.509" y="1.016" extent="1-16" drill="0.3048"/>
-<via x="12.319" y="1.016" extent="1-16" drill="0.3048"/>
 <wire x1="10.2616" y1="24.8648" x2="10.2616" y2="25.3492" width="0.1524" layer="1"/>
 <wire x1="10.2616" y1="25.3492" x2="10.0076" y2="25.6032" width="0.1524" layer="1"/>
@@
 <via x="37.084" y="5.588" extent="1-16" drill="0.3048"/>
 <via x="39.37" y="5.588" extent="1-16" drill="0.3048"/>
-<wire x1="12.319" y1="3.048" x2="12.319" y2="1.016" width="0" layer="19" extent="1-1"/>
 </signal>
 <signal name="SCL/SCK">
@@
 </signal>
 <signal name="!RESET">
-<wire x1="18.7452" y1="3.5052" x2="26.56765625" y2="3.5052" width="0.1524" layer="16"/>
 <via x="26.797" y="17.7546" extent="1-16" drill="0.3048"/>
 <wire x1="26.67" y1="17.6276" x2="26.67" y2="13.6906" width="0.1524" layer="16"/>
@@
 <wire x1="26.32" y1="18.7396" x2="26.32" y2="18.8306" width="0.1524" layer="1"/>
 <contactref element="JP15" pad="4"/>
-<wire x1="13.97" y1="1.27" x2="18.7452" y2="3.5052" width="0" layer="19" extent="16-16"/>
+<wire x1="13.97" y1="1.27" x2="26.56765625" y2="3.5052" width="0" layer="19" extent="16-16"/>
 </signal>
 <signal name="TXLV">
@@
 <wire x1="27.051" y1="2.794" x2="27.686" y2="3.429" width="0.1524" layer="16"/>
 <via x="27.813" y="3.429" extent="1-16" drill="0.3048"/>
-<wire x1="23.114" y1="2.794" x2="27.051" y2="2.794" width="0.1524" layer="16"/>
 <wire x1="30.353" y1="3.429" x2="27.813" y2="3.429" width="0.1524" layer="1"/>
 <wire x1="27.686" y1="3.429" x2="27.813" y2="3.429" width="0.1524" layer="16"/>
@@
 <wire x1="30.751" y1="12.5306" x2="26.32" y2="12.5306" width="0.1524" layer="1"/>
 <contactref element="JP15" pad="2"/>
-<wire x1="19.05" y1="1.27" x2="23.114" y2="2.794" width="0" layer="19" extent="16-16"/>
+<wire x1="19.05" y1="1.27" x2="27.051" y2="2.794" width="0" layer="19" extent="16-16"/>
 </signal>
 <signal name="PPS">
 <contactref element="PPS" pad="2"/>
 <via x="27.686" y="11.4046" extent="1-16" drill="0.3048"/>
-<wire x1="16.51" y1="3.81" x2="26.1181125" y2="3.81" width="0.1524" layer="16"/>
 <wire x1="33.2486" y1="10.8966" x2="32.385" y2="10.8966" width="0.1524" layer="16"/>
 <via x="32.385" y="10.8966" extent="1-16" drill="0.3048"/>
@@
 <wire x1="27.686" y1="11.4046" x2="27.686" y2="5.3778875" width="0.1524" layer="16"/>
 <contactref element="JP15" pad="5"/>
-<wire x1="11.43" y1="1.27" x2="16.51" y2="3.81" width="0" layer="19" extent="16-16"/>
+<wire x1="11.43" y1="1.27" x2="26.1181125" y2="3.81" width="0" layer="19" extent="16-16"/>
 </signal>
 <signal name="N$5">
@@
 </signal>
 <signal name="TP2/!SAFE">
-<wire x1="20.9042" y1="3.1242" x2="26.82165625" y2="3.1242" width="0.1524" layer="16"/>
 <wire x1="26.82165625" y1="3.1242" x2="29.0068" y2="5.30934375" width="0.1524" layer="16"/>
 <wire x1="28.4052875" y1="9.2306" x2="28.99064375" y2="8.64524375" width="0.1524" layer="1"/>
@@
 <wire x1="26.32" y1="9.2306" x2="28.4052875" y2="9.2306" width="0.1524" layer="1"/>
 <contactref element="JP15" pad="3"/>
-<wire x1="16.51" y1="1.27" x2="20.9042" y2="3.1242" width="0" layer="19" extent="16-16"/>
+<wire x1="16.51" y1="1.27" x2="26.82165625" y2="3.1242" width="0" layer="19" extent="16-16"/>
 </signal>
 <signal name="RXI/MOSI">
@@
 <signal name="SHLD">
 <polygon width="0.2032" layer="16">
-<vertex x="15.494" y="32.9946"/>
-<vertex x="15.494" y="26.6192"/>
-<vertex x="5.461" y="26.6192"/>
-<vertex x="5.461" y="32.9946"/>
+<vertex x="15.113" y="32.9946"/>
+<vertex x="15.113" y="26.6192"/>
+<vertex x="6.096" y="26.6192"/>
+<vertex x="6.096" y="32.9946"/>
 </polygon>
 <polygon width="0.2032" layer="1">
-<vertex x="15.494" y="32.9946"/>
-<vertex x="15.494" y="26.6192"/>
-<vertex x="5.461" y="26.6192"/>
-<vertex x="5.461" y="32.9946"/>
+<vertex x="15.113" y="32.9946"/>
+<vertex x="15.113" y="26.6192"/>
+<vertex x="5.969" y="26.6192"/>
+<vertex x="5.969" y="32.9946"/>
 </polygon>
 <via x="14.097" y="30.4546" extent="1-16" drill="0.3048"/>
@@
 <contactref element="U1" pad="2"/>
 <wire x1="26.32" y1="10.3306" x2="28.136" y2="10.3306" width="0.1524" layer="1"/>
-<contactref element="R16" pad="1"/>
 <contactref element="SPI" pad="2"/>
-<wire x1="29.6884" y1="11.0236" x2="29.718" y2="10.994" width="0.254" layer="1"/>
-<wire x1="28.829" y1="11.0236" x2="29.6884" y2="11.0236" width="0.1524" layer="1"/>
 <wire x1="28.8036" y1="9.8806" x2="28.8036" y2="10.9982" width="0.1524" layer="16"/>
 <wire x1="28.8036" y1="10.9982" x2="28.829" y2="11.0236" width="0.1524" layer="16"/>
